Commit message: Husky with UR5e

File: robot_models/husky/husky.urdf (robot description, URDF)
Before this commit: robot husky_robot, 11 links, 10 joints
Links:
- added link top_plate2_link; collision mesh filename=D:\Mobile Manipulator Research\manipulator_control\robot_mo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; visual mesh filename=D:\Mobile Manipulator Research\manipulator_control\robot_mo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
Joints:
- added joint top_plate2_joint: type fixed, parent base_link, child top_plate2_link, origin xyz=0.0812 0 0.245 rpy=0 0 0
